Commit message: 🚚 Rename line sensors links

File: urdf/colors.xacro (robot description, xacro)
@@ -25,17 +25,17 @@
     <material>Gazebo/Yellow</material>
   </gazebo>
-  <gazebo reference="sensor1_link">
+  <gazebo reference="line1_link">
     <material>Gazebo/Blue</material>
   </gazebo>
-  <gazebo reference="sensor2_link">
+  <gazebo reference="line2_link">
     <material>Gazebo/Blue</material>
   </gazebo>
-  <gazebo reference="sensor3_link">
+  <gazebo reference="line3_link">
     <material>Gazebo/Blue</material>
   </gazebo>
-  <gazebo reference="sensor4_link">
+  <gazebo reference="line4_link">
     <material>Gazebo/Blue</material>
   </gazebo>
-  <gazebo reference="sensor5_link">
+  <gazebo reference="line5_link">
     <material>Gazebo/Blue</material>
   </gazebo>

File: urdf/modelo_carrinho.urdf (robot description, URDF)
Before this commit: robot modelo_carrinho, 13 links, 12 joints
Links:
- removed link sensor1_link
- removed link sensor2_link
- removed link sensor3_link
- removed link sensor4_link
- removed link sensor5_link
- added link line1_link, mass 0.0011672687384539; collision mesh filename=package://modelo_carrinho/meshes/line1_link.stl; visual mesh filename=package://modelo_carrinho/meshes/line1_link.stl
- added link line2_link, mass 0.0011672687384539; collision mesh filename=package://modelo_carrinho/meshes/line2_link.stl; visual mesh filename=package://modelo_carrinho/meshes/line2_link.stl
- added link line3_link, mass 0.0011672687384539; collision mesh filename=package://modelo_carrinho/meshes/line3_link.stl; visual mesh filename=package://modelo_carrinho/meshes/line3_link.stl
- added link line4_link, mass 0.0011672687384539; collision mesh filename=package://modelo_carrinho/meshes/line4_link.stl; visual mesh filename=package://modelo_carrinho/meshes/line4_link.stl
- added link line5_link, mass 0.0011672687384539; collision mesh filename=package://modelo_carrinho/meshes/line5_link.stl; visual mesh filename=package://modelo_carrinho/meshes/line5_link.stl
Joints:
- removed joint sensor1_joint
- removed joint sensor2_joint
- removed joint sensor3_joint
- removed joint sensor4_joint
- removed joint sensor5_joint
- added joint line1_joint: type fixed, parent base_link, child line1_link, origin xyz=0.12967 0.03813 -0.024382 rpy=0 1.5708 0, axis 0 0 0
- added joint line2_joint: type fixed, parent base_link, child line2_link, origin xyz=0.12967 0.01893 -0.024382 rpy=0 1.5708 0, axis 0 0 0
- added joint line3_joint: type fixed, parent base_link, child line3_link, origin xyz=0.12967 -9E-05 -0.024382 rpy=0 1.5708 0, axis 0 0 0
- added joint line4_joint: type fixed, parent base_link, child line4_link, origin xyz=0.12967 -0.01911 -0.024382 rpy=0 1.5708 0, axis 0 0 0
- added joint line5_joint: type fixed, parent base_link, child line5_link, origin xyz=0.12967 -0.03795 -0.024382 rpy=0 1.5708 0, axis 1 0 0
