Commit message: Fix typo

File: urdf/modelo_carrinho.urdf (robot description, URDF)
Before this commit: robot modelo_carrinho, 13 links, 12 joints
Joints:
- removed joint rodaesqueda_joint
- added joint rodaesquerda_joint: type continuous, parent base_link, child rodaesquerda_link, origin xyz=0 0.0755 -0.0019934 rpy=0 0 0, axis 0 1 0

Commit message: Change meshes file extension

File: urdf/modelo_carrinho.urdf (robot description, URDF)
Before this commit: robot modelo_carrinho, 13 links, 12 joints
Links:
- link arduino_link: geometry collision mesh filename=package://modelo_carrinho/meshes/arduino_link.stl; visual mesh filename=package://modelo_carrinho/meshes/arduino_link.stl
- link base_link: geometry collision mesh filename=package://modelo_carrinho/meshes/base_link.stl; visual mesh filename=package://modelo_carrinho/meshes/base_link.stl
- link bateria_link: geometry collision mesh filename=package://modelo_carrinho/meshes/bateria_link.stl; visual mesh filename=package://modelo_carrinho/meshes/bateria_link.stl
- link motordireito_link: geometry collision mesh filename=package://modelo_carrinho/meshes/motordireito_link.stl; visual mesh filename=package://modelo_carrinho/meshes/motordireito_link.stl
- link motoresquerdo_link: geometry collision mesh filename=package://modelo_carrinho/meshes/motoresquerdo_link.stl; visual mesh filename=package://modelo_carrinho/meshes/motoresquerdo_link.stl
- link rodadireita_link: geometry collision mesh filename=package://modelo_carrinho/meshes/rodadireita_link.stl; visual mesh filename=package://modelo_carrinho/meshes/rodadireita_link.stl
- link rodaesquerda_link: geometry collision mesh filename=package://modelo_carrinho/meshes/rodaesquerda_link.stl; visual mesh filename=package://modelo_carrinho/meshes/rodaesquerda_link.stl
- link sensor1_link: geometry collision mesh filename=package://modelo_carrinho/meshes/sensor1_link.stl; visual mesh filename=package://modelo_carrinho/meshes/sensor1_link.stl
- link sensor2_link: geometry collision mesh filename=package://modelo_carrinho/meshes/sensor2_link.stl; visual mesh filename=package://modelo_carrinho/meshes/sensor2_link.stl
- link sensor3_link: geometry collision mesh filename=package://modelo_carrinho/meshes/sensor3_link.stl; visual mesh filename=package://modelo_carrinho/meshes/sensor3_link.stl
- link sensor4_link: geometry collision mesh filename=package://modelo_carrinho/meshes/sensor4_link.stl; visual mesh filename=package://modelo_carrinho/meshes/sensor4_link.stl
- link sensor5_link: geometry collision mesh filename=package://modelo_carrinho/meshes/sensor5_link.stl; visual mesh filename=package://modelo_carrinho/meshes/sensor5_link.stl
- link sonar_link: geometry collision mesh filename=package://modelo_carrinho/meshes/sonar_link.stl; visual mesh filename=package://modelo_carrinho/meshes/sonar_link.stl

Commit message: ♻️ Refactor model - Create other coordinate systems for each sensor mesh, so that the sensor plugin position can be easily configured
Co-authored-by: Lucas Haug <LucasHaug@users.noreply.github.com>
Co-authored-by: Thalles Carneiro <mr-coala@users.noreply.github.com>

File: urdf/modelo_carrinho.urdf (robot description, URDF)
Before this commit: robot modelo_carrinho, 13 links, 12 joints
Links:
- link rodadireita_link: mass 0.0293925354796174 -> 0.0293925354796178
Joints:
- joint rodadireita_joint: origin xyz=0 -0.076 0.0020066 rpy=0 0 0 -> xyz=0 -0.076 0 rpy=0 0 0
- joint rodaesquerda_joint: origin xyz=0 0.0755 -0.0019934 rpy=0 0 0 -> xyz=0 0.0755 0 rpy=0 0 0
- joint sensor1_joint: origin xyz=0 0 0 rpy=0 0 0 -> xyz=0.12967 0.03813 -0.024382 rpy=0 1.5708 0
- joint sensor2_joint: origin xyz=0 0 0 rpy=0 0 0 -> xyz=0.12967 0.01893 -0.024382 rpy=0 1.5708 0
- joint sensor3_joint: origin xyz=0 0 0 rpy=0 0 0 -> xyz=0.12967 -9E-05 -0.024382 rpy=0 1.5708 0
- joint sensor4_joint: origin xyz=0 0 0 rpy=0 0 0 -> xyz=0.12967 -0.01911 -0.024382 rpy=0 1.5708 0
- joint sensor5_joint: axis 0 0 0 -> 1 0 0; origin xyz=0 0 0 rpy=0 0 0 -> xyz=0.12967 -0.03795 -0.024382 rpy=0 1.5708 0
- joint sonar_joint: axis 0 1 0 -> 0 0 1; origin xyz=0 0 0 rpy=0 0 0 -> xyz=0.17102 0.00018254 -0.00125 rpy=1.5708 0 0; type prismatic -> fixed

Commit message: 🐛 Fix the joint axis direction so that positive angular velocity mean forward motion
Co-authored-by: Felipe Gomes de Melo <felipegmelo.42@gmail.com>

File: urdf/modelo_carrinho.urdf (robot description, URDF)
Before this commit: robot modelo_carrinho, 13 links, 12 joints
Joints:
- joint rodadireita_joint: axis 0 -1 0 -> 0 1 0; limit (none) -> effort=78e-3 velocity=15.0
- joint rodaesquerda_joint: limit (none) -> effort=78e-3 velocity=15.0

Commit message: ⏪ Undo limit config in urdf file

File: urdf/modelo_carrinho.urdf (robot description, URDF)
Before this commit: robot modelo_carrinho, 13 links, 12 joints
Joints:
- joint rodadireita_joint: limit effort=78e-3 velocity=15.0 -> (none)
- joint rodaesquerda_joint: limit effort=78e-3 velocity=15.0 -> (none)
